File: Circuits/Motor_Control/Motor_circuit_v1/Motor_circuit_v1.kicad_sch (KiCad schematic)
At the start: 0 parts

Commit message: motor circuit kicad, STSPIN32F0 with SQS mosfets
Parts:
- added Q1, Q2, Q3, Q4, Q5, Q6: SQS178ELNW-T1_GE3, POWERPAK_1212-8SLW_VIS, symbol SQS178ELNW-T1-GE3:SQS178ELNW-T1_GE3
- added U1: STSPIN32F0, VFQFPN48_7X7X1_STM, symbol STSPIN32F0:STSPIN32F0
Connections:
- new net: Q2.3, Q3.3, Q6.3
- new net: Q3.4, U1.36 (LSU)
- new net: Q1.3, Q3.8
- new net: Q1.4, U1.33 (HSU)
- new net: Q1.8, Q4.8, Q5.8
- new net: Q2.8, Q5.3
- new net: Q4.3, Q6.8

Commit message: Alternative motor driver circuit
Parts:
- removed U1: STSPIN32F0, VFQFPN48_7X7X1_STM, symbol STSPIN32F0:STSPIN32F0
- added Cbootu, Cbootv, Cbootw, Cbus, Ccs1, Ccs2, Clp, Creg, Cres, Cth, Cvdd: C, symbol Device:C
- added Cvdde, Cvm: C_Polarized, symbol Device:C_Polarized
- added Dhu, Dhv, Dhw, Dlu, Dlv, Dlw: D, symbol Device:D
- added J1: B5P-VH, CONN_B5P-VH_JST, symbol JST B5P-VH:B5P-VH
- added J2: B6B-PH-K-SLFSN, CONN_B6B-PH-K-S_JST, symbol JST B6B-PH-K-S:B6B-PH-K-SLFSN
- added J3: Conn_01x04_Pin, symbol Connector:Conn_01x04_Pin
- added NTC: Thermistor_NTC, symbol Device:Thermistor_NTC
- added R1, R2, R4, RH1, RH1m, RH1p, RH2, RH2m, RH2p, RH3, RH3m, RH3p, Rbus1, Rbus2, Rcs1, Rcs2, Rcs3, Rcs4, Rcs5, Rghu_off, Rghu_on, Rghv_off, Rghv_on, Rghw_off, Rghw_on, Rglu_off, Rglu_on, Rglv_off, Rglv_on, Rglw_off, Rglw_on, Rlp, Rs, Rth: R, symbol Device:R
- added R3: 1k, symbol Device:R
- added R5: 3k8, symbol Device:R
- added RESET: SW_Push, symbol Switch:SW_Push
- added U1: STSPIN32F0A, VFQFPN-48_7x7x1mm_STM, symbol STSPIN32F0A:STSPIN32F0A
Connections:
- net overcurrent_protection: now reaches Q3.1 (S)
- net overcurrent_protection: now also Q3.2 (S), Q3.3 (S), Q4.1 (S), Q4.2 (S), Q4.3 (S), Q6.1 (S), Q6.2 (S), Q6.3 (S), Rcs1.1, Rlp.1, Rs.1
- net at Q3.4 (G): now also Rglu_off.1, Rglu_on.1
- net OUTU: now reaches Q3.5 (D)
- net OUTU: now also Q1.1 (S), Q1.2 (S), Q1.3 (S), Q3.6 (D), Q3.7 (D), Q3.8 (D), Cbootu.2, J1.2 (Phase_U), U1.34 (OUTU)
- net at Q1.4 (G): now also Rghu_off.1, Rghu_on.1
- net VM: now reaches Q1.5 (D)
- net VM: now also Q1.6 (D), Q1.7 (D), Q1.8 (D), Q2.5 (D), Q2.6 (D), Q2.7 (D), Q2.8 (D), Q5.5 (D), Q5.6 (D), Q5.7 (D), Q5.8 (D), Cvm.1, Rbus1.1, U1.8 (VM)
- net OUTV: now reaches Q2.1 (S)
- net OUTV: now also Q2.2 (S), Q2.3 (S), Q4.5 (D), Q4.6 (D), Q4.7 (D), Q4.8 (D), Cbootv.2, J1.3 (Phase_V), U1.30 (OUTV)
- net at Q2.4 (G): now also Rghv_off.1, Rghv_on.1
- net OUTW: now reaches Q5.3 (S)
- net OUTW: now also Q5.1 (S), Q5.2 (S), Q6.5 (D), Q6.6 (D), Q6.7 (D), Q6.8 (D), Cbootw.2, J1.4 (Phase_W), U1.26 (OUTW); no longer Q2.8
- net at Q6.4 (G): now also Rglw_off.1, Rglw_on.1
- net at Q4.4 (G): now also Rglv_off.1, Rglv_on.1
- net at Q5.4 (G): now also Rghw_off.1, Rghw_on.1
- new net: Dlv.2 (A), Rglv_off.2
- new net: Dhu.2 (A), Rghu_off.2
- new net: Dlu.2 (A), Rglu_off.2
- new net: Dhw.2 (A), Rghw_off.2
- new net: Dhv.2 (A), Rghv_off.2
- new net: Dlw.2 (A), Rglw_off.2
- new net +2.5V: RH1m.2, RH2m.2, RH3m.2
- new net +5V: J2.2 (VCC(+5V)), R3.2, R5.1
- new net BOOT0: U1.42 (BOOT0)
- new net GND: Cbus.1, Ccs1.2, Clp.2, Creg.2, Cres.2, Cth.1, Cvdd.2, Cvdde.2, Cvm.2, J1.1 (GND), J1.5 (GND), J2.1 (GND), J2.6 (GND), NTC.2, R5.2, RESET.2, RH1p.2, RH2p.2, RH3p.2, Rbus2.2, Rcs3.2, Rcs4.2, Rs.2, U1.20 (TESTMODE), U1.44 (GND), U1.49 (EPAD)
- new net H1: J2.3 (Hall1), RH1.2
- new net H2: J2.4 (Hall2), RH2.2
- new net H3: J2.5 (Hall3), RH3.2
- new net HSU: Dhu.1 (K), Rghu_on.2, U1.33 (HSU)
- new net HSV: Dhv.1 (K), Rghv_on.2, U1.29 (HSV)
- new net HSW: Dhw.1 (K), Rghw_on.2, U1.25 (HSW)
- new net LSU: Dlu.1 (K), Rglu_on.2, U1.36 (LSU)
- new net LSV: Dlv.1 (K), Rglv_on.2, U1.32 (LSV)
- new net LSW: Dlw.1 (K), Rglw_on.2, U1.28 (LSW)
- new net NRST: Cres.1, RESET.1, U1.7 (NRST)
- new net OC_Comp: Clp.1, Rlp.2, U1.24 (OC_COMP)
- new net OP1N: Ccs2.2, Rcs4.1, Rcs5.2, U1.22 (OP1N)
- new net OP1O: Ccs2.1, Rcs5.1, U1.14 (PA3), U1.21 (OP1O)
- new net OP1P: Ccs1.1, Rcs1.2, Rcs2.2, Rcs3.1, U1.23 (OP1P)
- new net OP2N: R4.2, RH1.1
- new net OP2O: R4.1, U1.11 (PA0)
- new net OP2P: RH1m.1, RH1p.1
- new net OP3N: R1.2, RH2.1, U1.46 (OP3N)
- new net OP3O: R1.1, U1.12 (PA1), U1.47 (OP3O)
- new net OP3P: RH2m.1, RH2p.1, U1.45 (OP3P)
- new net OP4N: R2.2, RH3.1, U1.2 (OP2N)
- new net OP4O: R2.1, U1.13 (PA2), U1.3 (OP2O)
- new net OP4P: RH3m.1, RH3p.1, U1.1 (OP2P)
- new net PA13_SWD_IO: J3.2 (Pin_2), U1.37 (PA13_SWD_IO)
- new net PA14_SWD_CLK: J3.3 (Pin_3), U1.38 (PA14_SWD_CLK)
- new net PA15: U1.39 (PA15)
- new net PA4: U1.15 (PA4)
- new net PA5: Cbus.2, Rbus1.2, Rbus2.1, U1.16 (PA5)
- new net PA6: U1.17 (PA6)
- new net PA7: U1.18 (PA7)
- new net PB1: Cth.2, NTC.1, Rth.2, U1.19 (PB1)
- new net PB6: U1.40 (PB6)
- new net PB7: U1.41 (PB7)
- new net PF0: U1.4 (PF0)
- new net PF1: U1.5 (PF1)
- new net RESEREVED: U1.43 (RESERVED)
- new net SW: U1.9 (SW)
- new net VBOOTU: Cbootu.1, U1.35 (VBOOTU)
- new net VBOOTV: Cbootv.1, U1.31 (VBOOTV)
- new net VBOOTW: Cbootw.1, U1.27 (VBOOTW)
- new net VDD: Cvdd.1, Cvdde.1, Rcs2.1, Rth.1, U1.48 (VDD)
- new net VDDA: U1.10 (VDDA)
- new net VREG12: Creg.1, R3.1, U1.6 (VREG12)
Other:
- note added: "(output) (inverting input) (non-inverting input)"
- note added: "+24V Digital power supply"
- note added: "12 V linear regulator output"
- note added: "2.5 V"
- note added: "3.3 V DC/DC Buck regulator switching node (Analog out)"
- note added: "Analog voltage"
- note added: "Bus Voltage Measurement (VM) and Divider Network: The resistors RBUS1 and RBUS2, along with capacitor CBUS, form a voltage divider circuit connected to the main bus voltage (VM). Purpose: This circuit scales down the high bus voltage to a lower, measurable level suitable for the analog-to-digital converter (ADC) inputs of the microcontroller (PA5). The capacitor CBUS helps filter out high-frequen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"
- note added: "Capacitors (CBUS, CTH): CBUS and CTH are used for filtering purposes. They remove high-frequency noise and ensure that only the relevant low-frequency signals (representative of the bus voltage and temperature) are fed to the ADC."
- note added: "Capacitors (Ccs1, Ccs2) These capacitors are used for filtering. They smooth out high-frequency noise and ensure that the measured voltage accurately represents the current signal without interference from switching noise or other high-frequency disturbances."
- note added: "Connection to Overcurrent Comparator (OCCComp): After filtering and amplification, the conditioned signal is fed into the OCCComp comparator. This comparator compares the sensed current signal with a predefined threshold, which can be set using external resistors or by software. If the current exceeds the threshold, the comparator outputs a signal indicating an overcurrent condition."
- note added: "GND H3 H2 H1 +5V GND"
- note added: "GND W V U GND"
- note added: "Hall sensor 1 Feedback"
- note added: "Hall sensor 2 Feedback"
- note added: "Hall sensor 3 Feedback"
- note added: "Hall sensor connector"
- note added: "Internally connected to ground"
- note added: "Low-Pass Filter (RLP, CLP): This resistor and capacitor pair forms a low-pass filter, which removes high-frequency components from the sensed current signal. It ensures that only the average value or low-frequency components (representative of the actual current) are passed to the subsequent stages."
- note added: "Maybe unecessary"
- note added: "Motor connector"
- note added: "OpAmp inverting"
- note added: "OpAmp non-inverting"
- note added: "OpAmp output"
- note added: "Operational Amplifiers (OP0, OP1P, OP1N, OP1O, etc.): The operational amplifiers in the STSPIN32F0 are used to amplify and buffer the sensed current signal. They convert the differential voltage across the shunt resistor into a single-ended signal suitable for further processing."
- note added: "Output to ADC Input (PA3): The conditioned signal is also sent to an ADC input (PA3), allowing the microcontroller to monitor the current in real-time. This data can be used for feedback control or further processing in software."
- note added: "Overcurrent protection circuit"
- note added: "Phase U"
- note added: "Phase V"
- note added: "Phase W"
- note added: "Power supply voltage (bus voltage)"
- note added: "RESET"
- note added: "Reset"
- note added: "Resistors (RCS1, RCS2, RCS3, RCS4, RCS5): These resistors form part of a voltage divider network, conditioning the signal from the shunt resistor. This conditioning helps adjust the signal to a suitable range for the operational amplifiers and comparators within the STSPIN32F0."
- note added: "STSPIN32F0 Gate driver"
- note added: "Temperature Measurement Network (NTC and RTH): The NTC (Negative Temperature Coefficient thermistor) in conjunction with the resistor RTH forms a temperature sensing network. Purpose: This network provides real-time temperature feedback to the ADC input (PB1). As the temperature changes, the resistance of the NTC changes, altering the voltage at the ADC pin. This allows the microcontroller to mon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"
- note added: "Temperature measurement & signal conditioning"
- note added: "The resistor Rs is used to sense the current flowing through the circuit. The voltage drop across this resistor is proportional to the current, providing a measurable signal for the control system."
- note added: "VDD 24V Input"
- moved on the sheet: Q1, Q3
