File: Circuits/Mainboard/Mainboard/Mainboard.kicad_sch (KiCad schematic)
At the start: 46 parts, among them IC1 LM74500QDDFRQ1, IC2 LM74500QDDFRQ1, IC3 WSEN-ISDS 6-Dof IMU, IC4 SX1280IMLTRT, IC5 SKY66122-11, IC6 TS2596CM533_RNG, J1 XT60PW-M, J2 XT60PW-M, J3 Conn_01x07_Pin, J4 Conn_01x05_Pin, J5 B6B-PH-K-S, J6 B5P-VH_LF__SN_, J8 Conn_01x06_Pin, J9 Conn_01x05_Pin, Q1 PSMN6R7-40MLDX, Q2 PSMN6R7-40MLDX, U1 NUCLEOH723ZG

Commit message: Added components for mainboard
Parts:
- removed C11: 10uF, Capacitor_SMD:C_0805_2012Metric, symbol Device:C
- removed C8: 0.1uF, Capacitor_SMD:C_0805_2012Metric, symbol Device:C
- removed IC3: WSEN-ISDS 6-Dof IMU, WSEN-ISDS:2536030320001, symbol WSDN-ISDS:2536030320001
- removed J3: Conn_01x07_Pin, symbol Connector:Conn_01x07_Pin
- removed PS2: 5V Step down, 173010542, symbol FDSM 5V:173010542
- removed PS3: 12V Step down, 173011235, symbol FDSM 12V:173011235
- added C11, C8: 10uF, CAPC3225X280N, symbol 885012209073:885012209073
- added IC7: LM2576-5.0WU-TR, LM2576-5.0WU-TR:5-PIN-TO-263_U_, symbol LM2576-5.0WU-TR:LM2576-5.0WU-TR
- added J10, J12, J14, J16: B5P-VH_LF__SN_, B5P-VH-LF-SN:B5P-VH_LF__SN_, symbol B5P-VH-LF-SN:B5P-VH_LF__SN_
- added J11, J13, J7: B6B-PH-K-S, B6B-PH-K-S:JST_B6B-PH-K-S, symbol B6B-PH-K-S:B6B-PH-K-S
- added J3: Conn_01x06_Pin, symbol Connector:Conn_01x06_Pin
- C1, C3: footprint Capacitor_SMD:C_0805_2012Metric_Pad1.18x1.45mm_HandSolder -> CAPC2012X90N; symbol Device:C -> 885012207098:885012207098; Height (none) -> 0.9; Manufacturer_Name (none) -> Wurth Elektronik; Manufacturer_Part_Number (none) -> 885012207098; Mouser Part Number (none) -> 710-885012207098; Mouser Price/Stock (none) -> https://www.mouser.co.uk/ProductDetail/Wurth-Elektronik/885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
- C10, C9: footprint Capacitor_SMD:C_0805_2012Metric -> CAPC3225X280N; symbol Device:C -> 885012209073:885012209073; Height (none) -> 2.8; Manufacturer_Name (none) -> Wurth Elektronik; Manufacturer_Part_Number (none) -> 885012209073; Mouser Part Number (none) -> 710-885012209073; Mouser Price/Stock (none) -> https://www.mouser.co.uk/ProductDetail/Wurth-Elektronik/885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
- C12, C13, C14, C15, C17, C19, C2, C23, C4, C6, C7: footprint Capacitor_SMD:C_0805_2012Metric -> CAPC2012X90N; symbol Device:C -> 885012207098:885012207098; Height (none) -> 0.9; Manufacturer_Name (none) -> Wurth Elektronik; Manufacturer_Part_Number (none) -> 885012207098; Mouser Part Number (none) -> 710-885012207098; Mouser Price/Stock (none) -> https://www.mouser.co.uk/ProductDetail/Wurth-Elektronik/885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
- C16, C18: footprint Capacitor_SMD:C_0805_2012Metric -> CAPC2012X90N; symbol Device:C -> 885012007063:885012007063; Height (none) -> 0.9; Manufacturer_Name (none) -> Wurth Elektronik; Manufacturer_Part_Number (none) -> 885012007063; Mouser Part Number (none) -> 710-885012007063; Mouser Price/Stock (none) -> https://www.mouser.co.uk/ProductDetail/Wurth-Elektronik/885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
- C20, C21: footprint Capacitor_SMD:C_0805_2012Metric -> CAPC2012X90N; symbol Device:C -> 885012207092:885012207092; Height (none) -> 0.9; Manufacturer_Name (none) -> Wurth Elektronik; Manufacturer_Part_Number (none) -> 885012207092; Mouser Part Number (none) -> 710-885012207092; Mouser Price/Stock (none) -> https://www.mouser.co.uk/ProductDetail/Wurth-Elektronik/885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
- C22: footprint Capacitor_SMD:C_0805_2012Metric -> CAPAE1710X1700N; symbol Device:C_Polarized -> 865060663013:865060663013; Height (none) -> 17; Manufacturer_Name (none) -> Wurth Elektronik; Manufacturer_Part_Number (none) -> 865060663013; Mouser Part Number (none) -> 710-865060663013; Mouser Price/Stock (none) -> https://www.mouser.co.uk/ProductDetail/Wurth-Elektronik/865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
- C5: footprint Capacitor_SMD:C_0805_2012Metric -> CAPAE1030X1050N; symbol Device:C_Polarized -> 865080657018:865080657018; Height (none) -> 10.5; Manufacturer_Name (none) -> Wurth Elektronik; Manufacturer_Part_Number (none) -> 865080657018; Mouser Part Number (none) -> 710-865080657018; Mouser Price/Stock (none) -> https://www.mouser.co.uk/ProductDetail/Wurth-Elektronik/865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
Connections:
- net 24V: now also IC7.1 (VIN)
- net 24V_1: now also C8.1
- net 24V_2: now also C11.1
- net 3.3V: now also C13.2; no longer C13.1
- net BNO055_SCL: now also U1.CN12_3 (PB8)
- net BNO055_SDA: now also U1.CN11_21 (PB7)
- net GND: now also C13.1, C11.2, C8.2, IC7.3 (GND), IC7.5 (~{ON}/OFF), J3.1 (Pin_1); no longer C13.2
- net VL53L1_SCL: now also U1.CN11_51 (PF1)
- net VL53L1_SDA: now also U1.CN11_53 (PF0)
- net VL6180_SCL: now also U1.CN12_23 (PA8), J3.4 (Pin_4)
- net VL6180_SDA: now also U1.CN12_1 (PC9), J3.3 (Pin_3)
- net GND_LF: now reaches J5.1
- net GND_LF: now also J5.6
- net 5V_LF: now reaches J5.2
- net H1_LF: now reaches J5.3
- net H2_LF: now reaches J5.4
- net H3_LF: now reaches J5.5
- net Motor_GND: now reaches J6.1
- net Motor_GND: now also J6.5, J10.1, J10.5, J12.1, J12.5, J14.1, J14.5, J16.1, J16.5
- net U_LF: now reaches J6.2
- net V_LF: now reaches J6.3
- net W_LF: now reaches J6.4
- new net 2.8V: J3.2 (Pin_2)
- new net 5V_LR: J7.2
- new net 5V_RF: J11.2
- new net 5V_RR: J13.2
- new net GND_LR: J7.1, J7.6
- new net GND_RF: J11.1, J11.6
- new net GND_RR: J13.1, J13.6
- new net H1_LR: J7.3
- new net H1_RF: J11.3
- new net H1_RR: J13.3
- new net H2_LR: J7.4
- new net H2_RF: J11.4
- new net H2_RR: J13.4
- new net H3_LR: J7.5
- new net H3_RF: J11.5
- new net H3_RR: J13.5
- new net U_Dribbler: J16.2
- new net U_LR: J10.2
- new net U_RF: J12.2
- new net U_RR: J14.2
- new net VL6180_IO0: J3.5 (Pin_5)
- new net VL6180_IO1: J3.6 (Pin_6)
- new net V_Dribbler: J16.3
- new net V_LR: J10.3
- new net V_RF: J12.3
- new net V_RR: J14.3
- new net W_Dribbler: J16.4
- new net W_LR: J10.4
- new net W_RF: J12.4
- new net W_RR: J14.4
- no-connect marks 15 -> 14
Other:
- note added: "Motor Connector Left Front (from above)"
- note added: "Motor Connector Rear right (from above)"
- note added: "VL53L4CD"
- note removed: "TOF400C-VL53L1"
- moved on the sheet: IC4, IC5, U1A, U1B, U1C, U1D, U1E, U1F, U1G, U1H, U1I, U1J

Commit message: Added components for mainboard
Parts:
- added C24: 10uF, CAPC3225X280N, symbol 885012209073:885012209073
- added C25, C26: 0.1uF, CAPC2012X90N, symbol 885012207098:885012207098
- added IC3: 2536030320001, WSEN-ISDS:2536030320001, symbol WSEN-ISDS:2536030320001
- added J15: SMA-J-P-H-RA-TH1, SMA-J-P-H-RA-TH1:SMAJPHRATH1, symbol SMA-J-P-H-RA-TH1:SMA-J-P-H-RA-TH1
Connections:
- net 3.3V: now also C24.1, C25.1, IC3.8 (VDD)
- net GND: now also C24.2, C25.2, C26.2, IC3.6 (GND_1), IC3.7 (GND_2)
- net WSENS_CS: now reaches U1.CN11_32 (PA4)
- net WSENS_CS: now also IC3.12 (CS)
- net WSENS_SDA: now reaches U1.CN11_45 (PD7)
- net WSENS_SDA: now also IC3.14 (SDA)
- net WSENS_SCL: now reaches U1.CN12_11 (PA5)
- net WSENS_SCL: now also IC3.13 (SCL)
- net WSENS_SAO: now reaches U1.CN12_13 (PA6)
- net WSENS_SAO: now also IC3.1 (SAO)
- new net VDD_IO: C26.1, IC3.5 (VDD_IO)
- no-connect marks 14 -> 20
Other:
- note added: "WSENS-IMU"
- note added: "Wireless interface"
- moved on the sheet: C15, C16, C17, C18, C19, C20, C21, IC4, IC5

Commit message: Completet motor driver adapter board, added components for 3d rendering
Parts:
- removed IC7: LM2576-5.0WU-TR, LM2576-5.0WU-TR:5-PIN-TO-263_U_, symbol LM2576-5.0WU-TR:LM2576-5.0WU-TR
- removed J4: Conn_01x05_Pin, Connector_PinHeader_1.00mm:PinHeader_1x05_P1.00mm_Vertical, symbol Connector:Conn_01x05_Pin
- removed J9: Conn_01x05_Pin, symbol Connector:Conn_01x05_Pin
- added C27: 0.1uF, CAPC2012X90N, symbol 885012207098:885012207098
- added C28: 47uF, Altium_WCAP-CSGP (rev24b):WCAP-CSGP_0805_L2W1.25H1.25, symbol Altium_WCAP-CSGP (rev24b):885012107006
- added IC7: TPS563300DRLR, TPS563300DRLR:TPS62932DRLR, symbol TPS563300DRLR:TPS563300DRLR
- added J17, J18, J19, J20, J21: ~, 61301021821:ESC_Adapter_socket, symbol 61301021821:6130XX21821_61301021821
- added J22, J23, J24, J9: 61300211821, Socket_header_6_pins_single_straight:61300211821, symbol Socket_header_6_pins_single_straight:61300211821
- added J25: Conn_01x06_Pin, Socket_header_6_pins_single_straight:61300611821, symbol Socket_header_6_pins_single_straight:61300611821
- added J26: Conn_01x04_Pin, Connector_PinHeader_2.54mm:PinHeader_1x04_P2.54mm_Vertical, symbol Connector:Conn_01x04_Pin
- added J4: ~, 61301021821:61301021821, symbol 61301021821:6130XX21821_61301021821
- added L1: 8.2uH, WE-HCC (rev24a):WE-HCC_1210, symbol WE-HCC (rev24a):7443330820
- added R3: 52.3kOhm, CRCW060352K3FKEA:RESC1608X50N, symbol Altium_WRIS-RSKS (rev23a):560112120013
- added R4: 10kOhm, Altium_WRIS-RSKS (rev23a):WRIS-RSKS_0805_Wave, symbol Altium_WRIS-RSKS (rev23a):560112120004
- C22: footprint CAPAE1710X1700N -> Altium_WCAP-ASLL (rev24b):WCAP-ASLL_D16H17; symbol 865060663013:865060663013 -> Altium_WCAP-ASLL (rev24b):865060663013; Capacitance (none) -> 470uF; Capacitance Tolerance (none) -> +/-20%; Category (none) -> Aluminum Electrolytic Capacitors; ComponentLink1Description (none) -> Website Link; ComponentLink1URL (none) -> https://www.we-online.com/redexpert/article/865060663013?ad; ComponentLink2Description (none) -> Datasheet Link; ComponentLink2URL (none) -> https://www.we-online.com/redexpert/spec/865060663013?ad; Diameter (none) -> 16mm; Dissipation Factor (none) -> 12%; Endurance (none) -> 5000h; Height 17 -> 17mm; Leakage Current (none) -> 235uA; Manufacturer (none) -> Wurth Elektronik; Manufacturer Part Number (none) -> 865060663013; Match Code (none) -> WCAP-ASLL; Mount (none) -> Surface Mount; Operating Temperature Max (none) -> 105°C; Operating Temperature Min (none) -> -55°C; Packaging (none) -> Tape and Reel; Rated Voltage (DC) (none) -> 50V; Ripple Current (none) -> 1610mA; Technical Reference (none) -> ASEK170471M050DVCTHE000
- J3, J8: footprint (none) -> Socket_header_6_pins_single_straight:61300611821; symbol Connector:Conn_01x06_Pin -> Socket_header_6_pins_single_straight:61300611821; Category (none) -> Board-to-Board Connectors; ComponentLink1Description (none) -> Website Link; ComponentLink1URL (none) -> https://www.we-online.com/redexpert/article/61300611821?ad; ComponentLink2Description (none) -> Datasheet Link; ComponentLink2URL (none) -> https://www.we-online.com/redexpert/spec/61300611821?ad; Contact Resistance (none) -> 20mOhm; Gender (none) -> Socket Header; Manufacturer (none) -> Wurth Elektronik; Manufacturer Part Number (none) -> 61300611821; Match Code (none) -> WR-PHD; Mount (none) -> Through Hole; Number of Pins (none) -> 6; Number of Rows (none) -> 1; Operating Temperature Max (none) -> 125°C; Operating Temperature Min (none) -> -40°C; Orientation (none) -> Vertical; Packaging (none) -> Tray; Pitch (none) -> 2.54mm; Rated Current (none) -> 3A; Withstanding Voltage (none) -> 500V; Working Voltage (none) -> 250V
Connections:
- net 5V_LF is gone; now on net 5V: J5.2
- net 5V_LR is gone; now on net 5V: J7.2
- net 5V_RR is gone; now on net 5V: J13.2
- net GND_LF is gone; now on net GND: J5.1, J5.6
- net GND_LR is gone; now on net GND: J7.1, J7.6
- net GND_RF is gone; now on net GND: J11.1, J11.6
- net GND_RR is gone; now on net GND: J13.1, J13.6
- net H3_LF is gone; now on net M1_H3: J5.5
- net Motor_GND is gone; now on net GND: J10.1, J10.5, J12.1, J12.5, J14.1, J14.5, J16.1, J16.5, J6.1, J6.5
- net VL53L1_INT is gone; now on net GND: J8.5
- net VL53L1_SHUT is gone; now on net 3.3V: J8.6
- net W_RF is gone; now on net M3_OUT3: J12.4
- net 2.8V: now also J3.5; no longer J3.2 (Pin_2)
- net 24V: now also IC7.3 (VIN), J17.13 (R3), J17.14 (R4), J18.13 (R3), J18.14 (R4), J19.13 (R3), J19.14 (R4), J20.13 (R3), J20.14 (R4), J21.13 (R3), J21.14 (R4)
- net 3.3V: now also J25.3, J4.9; no longer J8.1 (Pin_1)
- net 5V: now also C28.2, J17.3 (L3), J17.4 (L4), J18.3 (L3), J18.4 (L4), J19.3 (L3), J19.4 (L4), J20.3 (L3), J20.4 (L4), J21.3 (L3), J21.4 (L4), J26.3 (Pin_3), L1.2, R3.2
- net GND: now also J3.6, C28.1, IC7.4 (GND), J17.1 (L1), J17.11 (R1), J17.12 (R2), J17.2 (L2), J18.1 (L1), J18.11 (R1), J18.12 (R2), J18.2 (L2), J19.1 (L1), J19.11 (R1), J19.12 (R2), J19.2 (L2), J20.1 (L1), J20.11 (R1), J20.12 (R2), J20.2 (L2), J21.1 (L1), J21.11 (R1), J21.12 (R2), J21.2 (L2), J25.2, J26.4 (Pin_4), J4.7, R4.1; no longer J3.1 (Pin_1), J8.2 (Pin_2)
- net VL6180_IO0: now also J3.2; no longer J3.5 (Pin_5)
- net VL6180_IO1: now also J3.1; no longer J3.6 (Pin_6)
- net VL6180_SCL: now also J3.3; no longer J3.4 (Pin_4)
- net VL6180_SDA: now also J3.4; no longer J3.3 (Pin_3)
- net M5_RX: now reaches U1.CN11_2 (PC11)
- net M5_RX: now also J21.7 (L7)
- net M5_TX: now reaches U1.CN11_28 (PA0)
- net M5_TX: now also J21.5 (L5)
- net Rpi_TX: now reaches U1.CN11_3 (PC12)
- net Rpi_TX: now also J26.1 (Pin_1)
- net M4_RX: now reaches U1.CN11_46 (PE2)
- net M4_RX: now also J20.7 (L7)
- net M4_TX: now reaches U1.CN11_47 (PE3)
- net M4_TX: now also J20.5 (L5)
- net Rpi_RX: now reaches U1.CN12_16 (PB12)
- net Rpi_RX: now also J26.2 (Pin_2)
- net M1_TX: now reaches U1.CN12_17 (PB6)
- net M1_TX: now also J17.5 (L5)
- net M3_RX: now reaches U1.CN12_19 (PC7)
- net M3_RX: now also J19.7 (L7)
- net M1_RX: now reaches U1.CN12_26 (PB15)
- net M1_RX: now also J17.7 (L7)
- net M2_TX: now reaches U1.CN12_35 (PA2)
- net M2_TX: now also J18.5 (L5)
- net M2_RX: now reaches U1.CN12_37 (PA3)
- net M2_RX: now also J18.7 (L7)
- net M3_TX: now reaches U1.CN12_4 (PC6)
- net M3_TX: now also J19.5 (L5)
- net ADPS-9960_SCL: now reaches U1.CN12_50 (PF14)
- net ADPS-9960_SCL: now also J25.5
- net ADPS-9960_SDA: now reaches U1.CN12_60 (PF15)
- net ADPS-9960_SDA: now also J25.4
- net BNO055_SCL renamed SEN0374_SCL
- net SEN0374_SCL: now also J4.5
- net BNO055_SDA renamed SEN0374_SDA
- net SEN0374_SDA: now also J4.3
- net H1_LF renamed M1_H3
- net M1_H3: now also J17.6 (L6)
- net H1_LR renamed M2_H1
- net M2_H1: now also J18.10 (L10)
- net H1_RF renamed M3_H1
- net M3_H1: now also J19.10 (L10)
- net H1_RR renamed M4_H1
- net M4_H1: now also J20.10 (L10)
- net H2_LF renamed M1_H2
- net M1_H2: now also J17.8 (L8)
- net H2_LR renamed M2_H2
- net M2_H2: now also J18.8 (L8)
- net H2_RF renamed M3_H2
- net M3_H2: now also J19.8 (L8)
- net H2_RR renamed M4_H2
- net M4_H2: now also J20.8 (L8)
- net H3_LR renamed M2_H3
- net M2_H3: now also J18.6 (L6)
- net H3_RF renamed M3_H3
- net M3_H3: now also J19.6 (L6)
- net H3_RR renamed M4_H3
- net M4_H3: now also J20.6 (L6)
- net U_Dribbler renamed M5_OUT1
- net M5_OUT1: now also J21.19 (R9), J21.20 (R10)
- net U_LF renamed M1_OUT1
- net M1_OUT1: now also J17.19 (R9), J17.20 (R10)
- net U_LR renamed M2_OUT1
- net M2_OUT1: now also J18.19 (R9), J18.20 (R10)
- net U_RF renamed M3_OUT3
- net M3_OUT3: now also J19.15 (R5), J19.16 (R6)
- net U_RR renamed M4_OUT1
- net M4_OUT1: now also J20.19 (R9), J20.20 (R10)
- net VL53L1_SCL renamed VL53L4CD_SCL
- net VL53L4CD_SCL: now also J8.3; no longer J8.4 (Pin_4)
- net VL53L1_SDA renamed VL53L4CD_SDA
- net VL53L4CD_SDA: now also J8.4; no longer J8.3 (Pin_3)
- net V_Dribbler renamed M5_OUT2
- net M5_OUT2: now also J21.17 (R7), J21.18 (R8)
- net V_LF renamed M1_OUT2
- net M1_OUT2: now also J17.17 (R7), J17.18 (R8)
- net V_LR renamed M2_OUT2
- net M2_OUT2: now also J18.17 (R7), J18.18 (R8)
- net V_RF renamed M3_OUT2
- net M3_OUT2: now also J19.17 (R7), J19.18 (R8)
- net V_RR renamed M4_OUT2
- net M4_OUT2: now also J20.17 (R7), J20.18 (R8)
- net W_Dribbler renamed M5_OUT3
- net M5_OUT3: now also J21.15 (R5), J21.16 (R6)
- net W_LF renamed M1_OUT3
- net M1_OUT3: now also J17.15 (R5), J17.16 (R6)
- net W_LR renamed M2_OUT3
- net M2_OUT3: now also J18.15 (R5), J18.16 (R6)
- net W_RR renamed M4_OUT3
- net M4_OUT3: now also J20.15 (R5), J20.16 (R6)
- new net: IC7.8 (FB), R3.1, R4.2
- new net: C27.1, IC7.5 (SW), L1.1
- new net: C27.2, IC7.6 (BST)
- new net ADPS-9960_INT: J25.6
- new net ADPS-9960_VL: J25.1
- new net M1_Encoder_A: J23.1
- new net M1_Encoder_B: J23.2
- new net M1_H1: J17.10 (L10)
- new net M1_PWM: J17.9 (L9)
- new net M2_Encoder_A: J22.1
- new net M2_Encoder_B: J22.2
- new net M2_PWM: J18.9 (L9)
- new net M3_Encoder_A: J24.1
- new net M3_Encoder_B: J24.2
- new net M3_OUT1: J19.19 (R9), J19.20 (R10)
- new net M3_PWM: J19.9 (L9)
- new net M4_Encoder_A: J9.1
- new net M4_Encoder_B: J9.2
- new net M4_PWM: J20.9 (L9)
- new net M5_PWM: J21.9 (L9)
- new net SEN0374_BL-IND: J4.8
- new net SEN0374_Boot: J4.2
- new net SEN0374_INT: J4.1
- new net SEN0374_PS1: J4.4
- new net SEN0374_PS2: J4.6
- new net SEN0374_RST: J4.10
- new net VL53L4CD_INT: J8.2
- new net VL53L4CD_SHUT: J8.1
- no-connect marks 20 -> 209
Other:
- note added: "24V: Power for 5 BLDC motors, 10A max for each"
- note added: "3.3V: Power for nucleo-h723zg, BNO055, VL53, VL6180, WSENS-IMU"
- note added: "5V: Power for raspberry pi 4 B 2A max"
- note added: "ADPS-9960"
- note added: "Motor 1"
- note added: "Motor 2"
- note added: "Motor 3"
- note added: "Motor 4"
- note added: "Motor 5 (dribbler)"
- note added: "Raspberry PI"
- note added: "SEN0374"
- note removed: "BNO055"
- note removed: "Motor Connector Left Front (from above)"
- note removed: "Motor Connector Rear right (from above)"
- moved on the sheet: C12, C13, C14, C15, C16, C17, C18, C19, C20, C21, C24, C25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
