File: Circuits/Mainboard/Mainboard/Mainboard.kicad_sch (KiCad schematic)
At the start: 71 parts, among them IC1 LM74500QDDFRQ1, IC2 LM74500QDDFRQ1, IC3 2536030320001, IC4 SX1280IMLTRT, IC5 SKY66122-11, IC6 TS2596CM533_RNG, IC7 TPS563300DRLR, J1 XT60PW-M, J10 B5P-VH_LF__SN_, J11 B6B-PH-K-S, J12 B5P-VH_LF__SN_, J13 B6B-PH-K-S, J14 B5P-VH_LF__SN_, J15 SMA-J-P-H-RA-TH1, J16 B5P-VH_LF__SN_, J2 XT60PW-M, J22 61300211821, J23 61300211821, J24 61300211821, J25 Conn_01x06_Pin, J26 Conn_01x04_Pin, J3 Conn_01x06_Pin, J5 B6B-PH-K-S, J6 B5P-VH_LF__SN_, J7 B6B-PH-K-S, J8 Conn_01x06_Pin, J9 61300211821, Q1 PSMN6R7-40MLDX, Q2 PSMN6R7-40MLDX, U1 NUCLEOH723ZG

Commit message: Step file for mainboard pcb updated layout
Parts:
- removed J22, J23, J24, J9: 61300211821, Socket_header_6_pins_single_straight:61300211821, symbol Socket_header_6_pins_single_straight:61300211821
- added J22, J23, J27, J9: Conn_01x04_Pin, Connector_PinHeader_2.54mm:PinHeader_1x04_P2.54mm_Vertical, symbol Connector:Conn_01x04_Pin
- J1, J2: footprint XT60PW-M:CONN_XT60PW-M_AMA -> Connector_AMASS:AMASS_XT60PW-M_1x02_P7.20mm_Horizontal
Connections:
- net 5V_RF is gone; now on net 5V: J11.2
- net 5V: now also J22.1 (Pin_1), J23.1 (Pin_1), J27.1 (Pin_1), J9.1 (Pin_1)
- net GND: now also J22.4 (Pin_4), J23.4 (Pin_4), J27.4 (Pin_4), J9.4 (Pin_4)
- net M1_Encoder_A: now also J22.2 (Pin_2)
- net M1_Encoder_B: now also J22.3 (Pin_3)
- net M2_Encoder_A: now also J9.2 (Pin_2)
- net M2_Encoder_B: now also J9.3 (Pin_3)
- net M3_Encoder_A: now also J23.2 (Pin_2)
- net M3_Encoder_B: now also J23.3 (Pin_3)
- net M4_Encoder_A: now also J27.2 (Pin_2)
- net M4_Encoder_B: now also J27.3 (Pin_3)
Other:
- moved on the sheet: IC5, J15

Commit message: Removed components from the pcb to make it easier to work with
Parts:
- C1, C12, C13, C14, C15, C16, C17, C18, C19, C2, C20, C21, C23, C25, C26, C27, C3, C4, C6, C7: footprint CAPC2012X90N -> 885012007063:CAPC2012X90N
- C10, C11, C24, C8, C9: footprint CAPC3225X280N -> 885012209073:CAPC3225X280N
- C5: footprint CAPAE1030X1050N -> 865080657018:CAPAE1030X1050N
Changed lines of the file:
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@@
 			)
 		)
-		(property "Footprint" "CAPC2012X90N"
+		(property "Footprint" "885012007063:CAPC2012X90N"
 			(at -55.55 187.96 0)
 			(effects
@@
 			)
 		)
-		(property "Footprint" "CAPC2012X90N"
+		(property "Footprint" "885012007063:CAPC2012X90N"
 			(at -12.37 106.68 0)
 			(effects
@@
 			)
 		)
-		(property "Footprint" "CAPC2012X90N"
+		(property "Footprint" "885012007063:CAPC2012X90N"
 			(at 512.14 78.74 0)
 			(effects
@@
 	)
 	(symbol
+		(lib_id "885012209073:885012209073")
+		(at 60.96 97.79 270)
+		(unit 1)
+		(exclude_from_sim no)
+		(in_bom yes)
+		(on_board yes)
+		(dnp no)
+		(property "Reference" "C8"
+			(at 56.134 99.314 90)
+			(effects
+				(font
+					(size 1.27 1.27)
+				)
+				(justify left)
+			)
+		)
+		(property "Value" "10uF"
+			(at 55.118 101.854 90)
+			(effects
+				(font
+					(size 1.27 1.27)
+				)
+				(justify left)
+			)
+		)
+		(property "Footprint" "885012209073:CAPC3225X280N"
+			(at -35.23 106.68 0)
+			(effects
+				(font
+					(size 1.27 1.27)
+				)
+				(justify left top)
+				(hide yes)
+			)
+		)
+		(property "Datasheet" "https://katalog.we-online.com/pbs/datasheet/885012209073.pdf"
+			(at -135.23 106.68 0)
+			(effects
+				(font
+					(size 1.27 1.27)
+				)
+				(justify left top)
+				(hide yes)
+			)
+		)
+		(property "Description" "Multilayer Ceramic Chip Capacitor WCAP-CSGP Series 1210 60pF X7R1210106K050DFCT10000"
+			(at 60.96 97.79 0)
+			(effects
+				(font
+					(size 1.27 1.27)
+				)
+				(hide yes)
+			)
+		)
+		(property "Height" "2.8"
+			(at -335.23 106.68 0)
+			(effects
+				(font
+					(size 1.27 1.27)
+				)
+				(justify left top)
+				(hide yes)
+			)
+		)
+		(property "Mouser Part Number" "710-885012209073"
+			(at -435.23 106.68 0)
+			(effects
+				(font
+					(size 1.27 1.27)
+				)
+				(justify left top)
+				(hide yes)
+			)
+		)
+		(property "Mouser Price/Stock" "https://www.mouser.co.uk/ProductDetail/Wurth-Elektronik/885012209073?qs=sPbYRqrBIVm8PsM2ljQIMg%3D%3D"
+			(at -535.23 106.68 0)
+			(effects
+				(font
+					(size 1.27 1.27)
+				)
+				(justify left top)
+				(hide yes)
+			)
+		)
+		(property "Manufacturer_Name" "Wurth Elektronik"
+			(at -635.23 106.68 0)
+			(effects
+				(font
+					(size 1.27 1.27)
+				)
+				(justify left top)
+				(hide yes)
+			)
+		)
+		(property "Manufacturer_Part_Number" "885012209073"
+			(at -735.23 106.68 0)
+			(effects
+				(font
+					(size 1.27 1.27)
+				)
+				(justify left top)
+				(hide yes)
+			)
+		)
+		(pin "1"
+		)
+		(pin "2"
+		)
+		(instances
+			(project "Mainboard"
+				(path "/778a7f39-1f28-457f-badd-61056e9c01e2"
+					(reference "C8")
+					(unit 1)
+				)
+			)
+		)
+	)
+	(symbol
 		(lib_id "power:GND")
 		(at 210.82 82.55 0)
@@
 			)
 		)
-		(property "Footprint" "CAPC2012X90N"
+		(property "Footprint" "885012007063:CAPC2012X90N"
 			(at -26.34 106.68 0)
 			(effects
@@
 			)
 		)
-		(property "Footprint" "CAPC2012X90N"
+		(property "Footprint" "885012007063:CAPC2012X90N"
 			(at -47.93 227.33 0)
 			(effects
@@
 			)
 		)
-		(property "Footprint" "CAPC2012X90N"
+		(property "Footprint" "885012007063:CAPC2012X90N"
 			(at 109.55 76.2 0)
 			(effects
@@
 			)
 		)
-		(property "Footprint" "CAPC3225X280N"
+		(property "Footprint" "885012209073:CAPC3225X280N"
 			(at 101.93 128.27 0)
 			(effects
@@
 			)
 		)
-		(property "Footprint" "CAPC2012X90N"
+		(property "Footprint" "885012007063:CAPC2012X90N"
 			(at -64.44 227.33 0)
 			(effects
@@
 	)
 	(symbol
-		(lib_id "885012209073:885012209073")
-		(at 60.96 97.79 270)
-		(unit 1)
-		(exclude_from_sim no)
-		(in_bom yes)
-		(on_board yes)
-		(dnp no)
-		(property "Reference" "C8"
-			(at 56.134 99.314 90)
-			(effects
-				(font
-					(size 1.27 1.27)
-				)
-				(justify left)
-			)
-		)
-		(property "Value" "10uF"
-			(at 55.118 101.854 90)
-			(effects
-				(font
-					(size 1.27 1.27)
-				)
-				(justify left)
-			)
-		)
-		(property "Footprint" "CAPC3225X280N"
-			(at -35.23 106.68 0)
-			(effects
-				(font
-					(size 1.27 1.27)
-				)
-				(justify left top)
-				(hide yes)
-			)
-		)
-		(property "Datasheet" "https://katalog.we-online.com/pbs/datasheet/885012209073.pdf"
-			(at -135.23 106.68 0)
-			(effects
-				(font
-					(size 1.27 1.27)
-				)
-				(justify left top)
-				(hide yes)
-			)
-		)
-		(property "Description" "Multilayer Ceramic Chip Capacitor WCAP-CSGP Series 1210 60pF X7R1210106K050DFCT10000"
-			(at 60.96 97.79 0)
-			(effects
-				(font
-					(size 1.27 1.27)
-				)
-				(hide yes)
-			)
-		)
-		(property "Height" "2.8"
-			(at -335.23 106.68 0)
-			(effects
-				(font
-					(size 1.27 1.27)
-				)
-				(justify left top)
-				(hide yes)
-			)
-		)
-		(property "Mouser Part Number" "710-885012209073"
-			(at -435.23 106.68 0)
-			(effects
-				(font
-					(size 1.27 1.27)
-				)
-				(justify left top)
-				(hide yes)
-			)
-		)
-		(property "Mouser Price/Stock" "https://www.mouser.co.uk/ProductDetail/Wurth-Elektronik/885012209073?qs=sPbYRqrBIVm8PsM2ljQIMg%3D%3D"
-			(at -535.23 106.68 0)
-			(effects
-				(font
-					(size 1.27 1.27)
-				)
-				(justify left top)
-				(hide yes)
-			)
-		)
-		(property "Manufacturer_Name" "Wurth Elektronik"
-			(at -635.23 106.68 0)
-			(effects
-				(font
-					(size 1.27 1.27)
-				)
-				(justify left top)
-				(hide yes)
-			)
-		)
-		(property "Manufacturer_Part_Number" "885012209073"
-			(at -735.23 106.68 0)
-			(effects
-				(font
-					(size 1.27 1.27)
-				)
-				(justify left top)
-				(hide yes)
-			)
-		)
-		(pin "1"
-		)
-		(pin "2"
-		)
-		(instances
-			(project "Mainboard"
-				(path "/778a7f39-1f28-457f-badd-61056e9c01e2"
-					(reference "C8")
-					(unit 1)
-				)
-			)
-		)
-	)
-	(symbol
 		(lib_id "B5P-VH-LF-SN:B5P-VH_LF__SN_")
 		(at 350.52 120.65 180)
@@
 			)
 		)
-		(property "Footprint" "CAPC2012X90N"
+		(property "Footprint" "885012007063:CAPC2012X90N"
 			(at 211.15 121.92 0)
 			(effects
@@
 			)
 		)
-		(property "Footprint" "CAPAE1030X1050N"
+		(property "Footprint" "865080657018:CAPAE1030X1050N"
 			(at 94.31 146.05 0)
 			(effects
@@
 			)
 		)
-		(property "Footprint" "CAPC2012X90N"
+		(property "Footprint" "885012007063:CAPC2012X90N"
 			(at -13.64 142.24 0)
 			(effects
@@
 			)
 		)
-		(property "Footprint" "CAPC2012X90N"
+		(property "Footprint" "885012007063:CAPC2012X90N"
 			(at 254 -23.8 0)
 			(effects
@@
 			)
 		)
-		(property "Footprint" "CAPC2012X90N"
+		(property "Footprint" "885012007063:CAPC2012X90N"
 			(at -56.82 227.33 0)
 			(effects
@@
 			)
 		)
-		(property "Footprint" "CAPC3225X280N"
+		(property "Footprint" "885012209073:CAPC3225X280N"
 			(at 498.17 78.74 0)
 			(effects
@@
 			)
 		)
-		(property "Footprint" "CAPC2012X90N"
+		(property "Footprint" "885012007063:CAPC2012X90N"
 			(at 9.22 231.14 0)
 			(effects
@@
 			)
 		)
-		(property "Footprint" "CAPC2012X90N"
+		(property "Footprint" "885012007063:CAPC2012X90N"
 			(at -40.31 227.33 0)
 			(effects
@@
 			)
 		)
-		(property "Footprint" "CAPC2012X90N"
+		(property "Footprint" "885012007063:CAPC2012X90N"
 			(at -45.39 187.96 0)
 			(effects
@@
 			)
 		)
-		(property "Footprint" "CAPC3225X280N"
+		(property "Footprint" "885012209073:CAPC3225X280N"
 			(at -36.5 142.24 0)
 			(effects
@@
 			)
 		)
-		(property "Footprint" "CAPC2012X90N"
+		(property "Footprint" "885012007063:CAPC2012X90N"
 			(at 109.55 128.27 0)
 			(effects
@@
 			)
 		)
-		(property "Footprint" "CAPC3225X280N"
+		(property "Footprint" "885012209073:CAPC3225X280N"
 			(at 101.93 76.2 0)
 			(effects
@@
 			)
 		)
-		(property "Footprint" "CAPC2012X90N"
+		(property "Footprint" "885012007063:CAPC2012X90N"
 			(at 524.84 325.12 0)
 			(effects
@@
 			)
 		)
-		(property "Footprint" "CAPC2012X90N"
+		(property "Footprint" "885012007063:CAPC2012X90N"
 			(at 453.72 90.17 0)
 			(effects
@@
 			)
 		)
-		(property "Footprint" "CAPC2012X90N"
+		(property "Footprint" "885012007063:CAPC2012X90N"
 			(at -26.34 142.24 0)
 			(effects
@@
 			)
 		)
-		(property "Footprint" "CAPC2012X90N"
+		(property "Footprint" "885012007063:CAPC2012X90N"
 			(at 306.4 300.99 0)
 			(effects
@@
 			)
 		)
-		(property "Footprint" "CAPC2012X90N"
+		(property "Footprint" "885012007063:CAPC2012X90N"
 			(at 624.51 337.82 0)
 			(effects
