File: Circuits/Mainboard/Mainboard/Mainboard.kicad_pcb (KiCad board)
At the start: 2 copper layers, 170 x 135.9 mm, 66 parts, among them IC1 LM74500QDDFRQ1, IC2 LM74500QDDFRQ1, IC3 2536030320001, IC6 TPS563300DRLR, IC7 TPS563300DRLR, J1 XT60PW-M, J10 B5P-VH_LF__SN_, J11 B6B-PH-K-S, J12 B5P-VH_LF__SN_, J13 B6B-PH-K-S, J14 B5P-VH_LF__SN_, J16 B5P-VH_LF__SN_, J17 Conn_01x04_Pin, J2 XT60PW-M, J23 Conn_01x04_Pin, J24 Conn_01x06_Pin, J25 Conn_01x06_Pin, J26 Conn_01x04_Pin, J27 Conn_01x04_Pin, J3 Conn_01x06_Pin, J5 B6B-PH-K-S, J6 B5P-VH_LF__SN_, J7 B6B-PH-K-S, J8 Conn_01x06_Pin, J9 Conn_01x04_Pin, P1 66200621122, Q1 PSMN6R7-40MLDX, Q2 PSMN6R7-40MLDX, U1 NUCLEOH723ZG, U2 ADP121-AUJZ28R7

Commit message: Exported mainboard, carrier board, and encoder to gerber
Parts:
- removed P1: 66200621122, WR-MPC3 3.00 mm Male Header Dual Row Vertical:66200621122
Routing:
- net GND: track 401.2 -> 228.3 mm, vias 48 -> 34
- net 24V: track 155.5 -> 76.6 mm, vias 19 -> 31
- net /VL53L4CD_INT: track 106.3 -> 132.8 mm
- net /M4_RX: track 95.1 -> 114.6 mm
- net /M3_Encoder_A: track 136.0 -> 150.0 mm, vias 1 -> 3
- net 3.3V: track 231.7 -> 242.5 mm, vias 3 -> 5
- net /M2_PWM: track 163.3 -> 173.2 mm, vias 5 -> 7
- net 2.8V: track 104.6 -> 96.6 mm
- net /ADPS-9960_SCL: track 111.8 -> 118.6 mm
- net /Rpi_RX: track 109.8 -> 115.7 mm, vias 2 -> 4
- net /VL6180_IO1: track 94.0 -> 99.6 mm, vias 5 -> 3
- net /ADPS-9960_VL: track 111.8 -> 116.9 mm
- net /M1_TX: track 103.3 -> 108.3 mm
- net /ADPS-9960_INT: track 113.3 -> 118.3 mm
- net /SEN0374_BL-IND: track 108.2 -> 113.1 mm, vias 4 -> 6
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
Commit message: Exported mainboard, carrier board, and encoder to gerber
Routing:
- net 3.3V: track 242.5 -> 243.5 mm
- net /VL6180_SCL: track 122.5 -> 123.5 mm
- net /M4_Encoder_B: track 68.4 -> 67.6 mm
- net /M5_RX: track 86.3 -> 86.9 mm
Other:
- board text added: "Motor 1"
- board text added: "Motor 2"
- board text added: "Motor 3"
- board text added: "Motor 4"
- board text added: "Motor 5"
- board text removed: "24V"
- board text removed: "OUT1"
- board text removed: "OUT2"
- board text removed: "OUT3"
