File: Circuits/Kicker_Control/KickerDesign/KickerCircuit_v.01.kicad_sch (KiCad schematic)
At the start: 9 parts, among them J1 Solenoid, Q1 NMOS, U1 NSL-32

Commit message: Version 2 of kicker.
Parts:
- removed D1, D2: 1N4148WT, Diode_SMD:D_SOD-523, symbol Diode:1N4148WT
- removed D3: 1.5KExxA, Diode_THT:D_DO-201AE_P15.24mm_Horizontal, symbol Diode:1.5KExxA
- removed U1: NSL-32, OptoDevice:Luna_NSL-32, symbol Isolator:NSL-32
- added D1: SMAJ20A, Diode_SMD:D_SMA, symbol Diode:SMAJ20A
- added D2: TLP3910_C20-TP,E, SOIC127P1000X220-6N, symbol TLP3910_C20-TP_E:TLP3910_C20-TP,E
- added U2, U3: VS-5EWH06FN-M3, DPAK_06FN-M3_VIS, symbol VS-5EWH06FN-M3:VS-5EWH06FN-M3
Connections:
- net Battery_In: now also U2.3
- net CVDC/V_OUT: now also U3.3
- net GND: now also D1.2 (A2), D2.3 (CATHODE_(INPUT))
- net On_signal/Off_signal: now also D2.1 (ANODE_(INPUT))
- net at C1.1, Q1.2 (G), R2.2: now also D1.1 (A1)
- net at J1.2 (Pin_2), Q1.1 (D): now also U3.2
- net at R1.1, R2.1: now also D2.4 (CATHODE_(OUTPUT)_1)
- new net: D2.6 (ANODE_(OUTPUT)), U2.2
